File: PCB/venkat-pcb.kicad_pcb (KiCad board)
At the start: 2 copper layers, 11 parts, among them J1 Conn_01x03

Commit message: Update
Routing:
- added copper zone on F.Cu, net (none)
Other:
- board outline added: 102.5 x 18.5 mm
Changed lines of the file:
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@@
 			(outputformat 1)
 			(mirror no)
-			(drillshape 1)
+			(drillshape 0)
 			(scaleselection 1)
-			(outputdirectory "")
+			(outputdirectory "../Outputs PCB's/LED CLOCK - V1")
 		)
 	)
@@
 	)
 	(gr_line
-		(start 192.469672 107.57)
-		(end 192.469672 87.57)
+		(start 89 106.5)
+		(end 191.5 106.5)
 		(stroke
-			(width 0.2)
+			(width 0.05)
 			(type default)
 		)
-		(layer "Dwgs.User")
+		(layer "Edge.Cuts")
 	)
 	(gr_line
-		(start 87.46967 87.57)
-		(end 87.46967 107.57)
+		(start 191.5 88)
+		(end 89 88)
 		(stroke
-			(width 0.2)
+			(width 0.05)
 			(type default)
 		)
-		(layer "Dwgs.User")
+		(layer "Edge.Cuts")
 	)
 	(gr_line
-		(start 192.469672 87.57)
-		(end 87.46967 87.57)
+		(start 191.5 106.5)
+		(end 191.5 88)
 		(stroke
-			(width 0.2)
+			(width 0.05)
 			(type default)
 		)
-		(layer "Dwgs.User")
+		(layer "Edge.Cuts")
 	)
 	(gr_line
-		(start 87.46967 107.57)
-		(end 192.469672 107.57)
+		(start 89 88)
+		(end 89 106.5)
 		(stroke
-			(width 0.2)
+			(width 0.05)
 			(type default)
 		)
-		(layer "Dwgs.User")
+		(layer "Edge.Cuts")
 	)
 	(gr_text "S"
@@
 	)
 	(segment
-		(start 138 94.5)
-		(end 147 94.5)
+		(start 120 94.5)
+		(end 129 94.5)
 		(width 0.2)
 		(layer "F.Cu")
@@
 	)
 	(segment
-		(start 120 94.5)
-		(end 129 94.5)
+		(start 147 94.5)
+		(end 156 94.5)
 		(width 0.2)
 		(layer "F.Cu")
@@
 	)
 	(segment
-		(start 102.341722 94.5)
-		(end 111 94.5)
+		(start 165 94.5)
+		(end 174 94.5)
 		(width 0.2)
 		(layer "F.Cu")
@@
 	)
 	(segment
-		(start 165 94.5)
-		(end 174 94.5)
+		(start 102 94.670861)
+		(end 110.829139 94.670861)
 		(width 0.2)
 		(layer "F.Cu")
@@
 	)
 	(segment
-		(start 174 94.5)
-		(end 183 94.5)
+		(start 110.829139 94.670861)
+		(end 111 94.5)
 		(width 0.2)
 		(layer "F.Cu")
@@
 	)
 	(segment
-		(start 147 94.5)
-		(end 156 94.5)
+		(start 93 95)
+		(end 93.329139 94.670861)
 		(width 0.2)
 		(layer "F.Cu")
@@
 	)
 	(segment
-		(start 129 94.5)
-		(end 138 94.5)
+		(start 93.329139 94.670861)
+		(end 102 94.670861)
 		(width 0.2)
 		(layer "F.Cu")
@@
 	)
 	(segment
-		(start 165 94.5)
-		(end 156 94.5)
+		(start 111 94.5)
+		(end 120 94.5)
 		(width 0.2)
 		(layer "F.Cu")
@@
 	)
 	(segment
-		(start 102.170861 94.670861)
-		(end 102.341722 94.5)
+		(start 138 94.5)
+		(end 147 94.5)
 		(width 0.2)
 		(layer "F.Cu")
@@
 	)
 	(segment
-		(start 102 94.670861)
-		(end 102.170861 94.670861)
+		(start 174 94.5)
+		(end 183 94.5)
 		(width 0.2)
 		(layer "F.Cu")
@@
 	)
 	(segment
-		(start 111 94.5)
-		(end 120 94.5)
+		(start 92.91 94.91)
+		(end 93 95)
+		(width 0.2)
+		(layer "F.Cu")
+		(net 11)
+	)
+	(segment
+		(start 156 94.5)
+		(end 165 94.5)
 		(width 0.2)
 		(layer "F.Cu")
@@
 	(segment
 		(start 92.7 94.91)
-		(end 101.760861 94.91)
+		(end 92.91 94.91)
 		(width 0.2)
 		(layer "F.Cu")
@@
 	)
 	(segment
-		(start 101.760861 94.91)
-		(end 102 94.670861)
+		(start 129 94.5)
+		(end 138 94.5)
 		(width 0.2)
 		(layer "F.Cu")
@@
 		(net 12)
 	)
-	(group ""
-		(members "10789567-31fc-461d-bf3d-e0afaefbe87a" "4704a8db-215b-4477-8201-477c1d62ebce"
-			"63db7224-2282-4496-9d25-ddf30c9d9f25" "6f512abc-ed09-4d82-a2df-45944ba51f85"
+	(zone
+		(net 0)
+		(net_name "")
+		(layer "F.Cu")
+		(hatch edge 0.5)
+		(connect_pads
+			(clearance 0.5)
+		)
+		(min_thickness 0.25)
+		(filled_areas_thickness no)
+		(fill yes
+			(thermal_gap 0.5)
+			(thermal_bridge_width 0.5)
+			(island_removal_mode 1)
+			(island_area_min 10)
+		)
+		(polygon
+			(pts
+				(xy 195 85) (xy 85 85) (xy 85 110) (xy 195 110)
+			)
 		)
 	)

Commit message: Update
Parts:
- added H1: MountingHole, MountingHole:MountingHole_3.2mm_M3, F.Cu at (186.6, 90.5)
- added H2: MountingHole, MountingHole:MountingHole_3.2mm_M3, F.Cu at (125.8, 103.9)
- added J2: Conn_01x03, Connector_PinHeader_2.54mm:PinHeader_1x03_P2.54mm_Vertical, F.Cu at (190.4, 95.2)
Connections:
- D10 pad 2: unconnected-(D10-DOUT-Pad2) -> Net-(D10-DOUT)
Routing:
- net +5V: track 91.7 -> 0.00 mm
- net GND: track 90.5 -> 0.80 mm, vias 0 -> 315
- added copper zone on F.Cu, net +5V
- added copper zone on B.Cu, net GND
- added copper zone on F.Cu, net GND
- removed copper zone on F.Cu, net (none)
Other:
- board size 102.5 x 18.5 mm -> 103.9 x 18.5 mm
