File: PCB/venkat-pcb.kicad_sch (KiCad schematic)
At the start: 11 parts, among them J1 Conn_01x03

Commit message: Update
Parts:
- added H1, H2: MountingHole, MountingHole:MountingHole_3.2mm_M3, symbol Mechanical:MountingHole
- added J2: Conn_01x03, Connector_PinHeader_2.54mm:PinHeader_1x03_P2.54mm_Vertical, symbol Connector_Generic:Conn_01x03
Connections:
- net +5V: now also J2.3 (Pin_3)
- net GND: now also J2.1 (Pin_1)
- net at D10.2 (DOUT): now also J2.2 (Pin_2)
